File: PCB/Artnet_DMX_Converter/DMX.kicad_sch (KiCad schematic)
At the start: 45 parts, among them J10 XLR5, J11 XLR3, J4 XLR5, J5 XLR3, J6 XLR5, J7 XLR3, J8 XLR5, J9 XLR3, U10 MAX3485, U11 MAX3485, U12 TXS0101DCK, U8 MAX3485, U9 MAX3485

Commit message: Updated KiCad
Other:
- title: (none) -> GrandNA3_4Port_Node
Changed lines of the file:
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@@
 	(generator_version "9.0")
 	(paper "A4")
+	(title_block
+		(title "GrandNA3_4Port_Node")
+	)
 	(rectangle
 		(start 22.225 22.225)
