File: PCB/Artnet_DMX_Converter/POWER.kicad_sch (KiCad schematic)
At the start: 18 parts, among them IC1 NPM1300-QEAA-R7

Commit message: Updated KiCad
Other:
- title: (none) -> GrandNA3_4Port_Node
Changed lines of the file:
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@@
 	(generator_version "9.0")
 	(paper "A4")
+	(title_block
+		(title "GrandNA3_4Port_Node")
+	)
 	(junction
 		(at 99.06 137.16)
