File: PCB/Artnet_DMX_Converter/USB.kicad_sch (KiCad schematic)
At the start: 3 parts, among them J2 USB_C_Receptacle_USB2.0_14P, U3 USBLC6-2SC6

Commit message: Updated KiCad
Other:
- title: (none) -> GrandNA3_4Port_Node
Changed lines of the file:
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@@
 	(generator_version "9.0")
 	(paper "A4")
+	(title_block
+		(title "GrandNA3_4Port_Node")
+	)
 	(junction
 		(at 102.87 88.9)
