File: PCB/Artnet_DMX_Converter/WIFI.kicad_sch (KiCad schematic)
At the start: 1 part, among them J13 Conn_02x04

Commit message: Updated KiCad
Other:
- title: (none) -> GrandNA3_4Port_Node
Changed lines of the file:
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@@
 	(generator_version "9.0")
 	(paper "A4")
+	(title_block
+		(title "GrandNA3_4Port_Node")
+	)
 	(junction
 		(at 148.59 82.55)
