File: PCB/Artnet_DMX_Converter/Ethernet.kicad_sch (KiCad schematic)
At the start: 90 parts, among them J3 RJ45, T1 FA2805, U4 W5500, U5 VO618A-3X017T, U6 SI3402-B-GMR, U7 TLV431, Y2 ABM8-25.000MHZ-10-D1G-T

Commit message: Updated KiCad
Other:
- title: (none) -> GrandNA3_4Port_Node
Changed lines of the file:
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@@
 	(generator_version "9.0")
 	(paper "A4")
+	(title_block
+		(title "GrandNA3_4Port_Node")
+	)
 	(junction
 		(at 217.17 38.1)

Commit message: Updated pcb files again....
Parts:
- U5: value VO618A-3X017T -> VO618A-3X019T
- Y2: private KLC_S4.1 -> (none)
Changed lines of the file:
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@@
-			)
-		)
-		(property private "KLC_S3.3" "The rectangle is not a symbol body but a graphical element"
-			(at 27.94 68.58 0)
-			(show_name yes)
-			(effects
-				(font
-					(size 1.27 1.27)
-				)
-				(hide yes)
-			)
-		)
-		(property private "KLC_S4.1" "Some pins are on 50mil grid to make the symbol small"
-			(at 27.94 66.04 0)
-			(show_name yes)
-			(effects
-				(font
-					(size 1.27 1.27)
-				)
-				(hide yes)
 			)
 		)
@@
 			)
 		)
-		(property "Value" "VO618A-3X017T"
+		(property "Value" "VO618A-3X019T"
 			(at 241.3 135.636 0)
 			(effects
