File: PCB/Artnet_DMX_Converter/Microcontroller.kicad_sch (KiCad schematic)
At the start: 34 parts, among them J1 Conn_01x03_MountingPin, SW1 SW_Push, SW2 SW_Push, U1 RP2350B, U2 W25Q128JVS, Y1 ABM8-272-T3

Commit message: Updated KiCad
Other:
- title: (none) -> GrandNA3_4Port_Node
Changed lines of the file:
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@@
 	(generator_version "9.0")
 	(paper "A4")
+	(title_block
+		(title "GrandNA3_4Port_Node")
+	)
 	(circle
 		(center 55.88 59.055)

Commit message: Updated pcb files again....
Parts:
- U1: private KLC_S4.2_VREG_LX -> (none)
- Y1: private KLC_S4.1 -> (none)
Changed lines of the file:
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@@
-			)
-		)
-		(property private "KLC_S4.2_DVDD" "Not a standalone power converter; internal on-chip voltage regulator for digital core supply; DVDD is the digital core power supply, should be placed next to voltage regulator output."
-			(at 146.05 100.33 0)
-			(show_name yes)
-			(effects
-				(font
-					(size 1.27 1.27)
-				)
-				(hide yes)
-			)
-		)
-		(property private "KLC_S4.2_VREG_LX" "Should be placed next to DVDD."
-			(at 146.05 100.33 0)
-			(show_name yes)
-			(effects
-				(font
-					(size 1.27 1.27)
-				)
-				(hide yes)
 			)
 		)
@@
 			(effects
 				(font
-					(size 1.27 1.27)
-				)
-				(hide yes)
-			)
-		)
-		(property private "KLC_S3.3" "The rectangle is not a symbol body but a graphical element"
-			(at 49.53 116.84 0)
-			(show_name yes)
-			(effects
-				(font
-					(size 1.27 1.27)
-				)
-				(hide yes)
-			)
-		)
-		(property private "KLC_S4.1" "Some pins are on 50mil grid to make the symbol small"
-			(at 46.99 116.84 0)
-			(show_name yes)
-			(effects
-				(font
